File: Fami_GITS2/Fami_GITS2.kicad_pcb (KiCad board)
At the start: 2 copper layers, 90.2 x 39.7 mm, 3 parts, among them J1 Famicom_Cartridge, U1 27C64, U2 27C64

Commit message: Completed schematic. PCB complete without routing.
Parts:
- added C1: 100 nF, Capacitor_THT:C_Disc_D3.0mm_W1.6mm_P2.50mm, F.Cu at (115.8, 100.2)
- added SW1: SW_SPDT, Button_Switch_SMD:SW_SPDT_CK-JS102011SAQN, F.Cu at (85.5, 86.4)
- added SW2: SW_SPDT, Button_Switch_SMD:SW_SPDT_CK-JS102011SAQN, F.Cu at (132.1, 86.4)
- added SW3: SW_SPDT, Button_Switch_SMD:SW_SPDT_CK-JS102011SAQN, F.Cu at (146.5, 86.4)
Connections:
- J1 pad 14: /CSS -> //CSS
- U1 pad 23: /A11 -> /IA11
- U2 pad 14: unconnected-(U2-GND-Pad14) -> GND
- U2 pad 21: /VA10 -> /IVA10
- U2 pad 23: /VA11 -> /IVA11
Routing:
- net VCC: track 130.4 -> 0.00 mm
- net /VA10: track 80.7 -> 0.00 mm
- net GND: track 73.9 -> 0.00 mm
- net //CSV: track 44.4 -> 0.00 mm
- net /A10: track 31.0 -> 0.00 mm
- net /A11: track 29.8 -> 0.00 mm
- net /D3: track 28.4 -> 0.00 mm
- net /D5: track 28.4 -> 0.00 mm
- net /D7: track 28.4 -> 0.00 mm
- net /D6: track 28.4 -> 0.00 mm
- net /D4: track 28.4 -> 0.00 mm
- net //OEV: track 27.3 -> 0.00 mm
- net /A9: track 26.4 -> 0.00 mm, vias 1 -> 0
- net /VA8: track 26.3 -> 0.00 mm, vias 1 -> 0
- net /VA11: track 26.2 -> 0.00 mm, vias 1 -> 0
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Other:
- board size 90.2 x 39.7 mm -> 90.2 x 49.9 mm
