File: Fami_GITS2/Fami_GITS2.kicad_sch (KiCad schematic)
At the start: 7 parts, among them J1 Famicom_Cartridge, SW1 SW_SPDT, SW2 SW_SPDT, SW3 SW_SPDT, U1 27C64, U2 27C64

Commit message: Completed schematic. PCB complete without routing.
Parts:
- C1: value C -> 100 nF; footprint (none) -> Capacitor_THT:C_Disc_D3.0mm_W1.6mm_P2.50mm
- SW1, SW2, SW3: footprint (none) -> Button_Switch_SMD:SW_SPDT_CK-JS102011SAQN
Connections:
- net CSS is gone; now on net /CSS: J1.14 (Pin_14)
- net A11: now also SW1.3 (C); no longer U1.23 (A11)
- net GND: now also C1.1, U2.14 (GND)
- net VA10: now also SW3.2 (B); no longer U2.21 (A10)
- net VA11: now also SW2.3 (C), SW3.3 (C); no longer U2.23 (A11)
- net VCC: now also C1.2, SW1.1 (A), SW2.1 (A)
- net IVA10: now reaches SW3.1 (A)
- net IVA10: now also U2.21 (A10)
- net IA11: now reaches SW1.2 (B)
- net IA11: now also U1.23 (A11)
- net IVA11: now reaches SW2.2 (B)
- net IVA11: now also U2.23 (A11)
Other:
- moved on the sheet: C1, J1, SW1, SW2, SW3
